Commit message: URDF Update

File: jaka_k1_ros2/src/jaka_k1_description/k1-de/urdf/jaka_k1.urdf (robot description, URDF)
Before this commit: robot jaka_k1, 20 links, 19 joints
Joints:
- joint rb2_j1: origin xyz=0 0 0 rpy=0 0 1.5708 -> xyz=0 0 0 rpy=0 0 -1.5708
- joint rb2_j3: axis 0 0 1 -> 0 0 -1; origin xyz=0 0 0 rpy=1.5708 0 3.1416 -> xyz=0 0 0 rpy=-1.5708 0 0
